Commit message: Adjust shape

File: src/fifth_robot_description/fifth_robot.urdf (robot description, URDF)
Before this commit: robot fifth_robot, 5 links, 4 joints
Links:
- link base_link: geometry collision box size=0.300 0.250 0.10; visual box size=0.300 0.250 0.10
- link caster_link: geometry collision sphere radius=0.07; visual sphere radius=0.07
- link left_wheel_link: geometry collision cylinder length=0.03 radius=0.07; visual cylinder length=0.03 radius=0.07
- link right_wheel_link: geometry collision cylinder length=0.03 radius=0.07; visual cylinder length=0.03 radius=0.07
Joints:
- joint caster_joint: origin xyz=0.150 0 -0.050 -> xyz=-0.200 0  0
- joint left_wheel_joint: axis 0 0 1 -> 0 0 -1; origin xyz=-0.100 0.130 0 rpy=-1.5707 0 0 -> xyz=0.136 -0.130 0 rpy=1.5707 0 0
- joint right_wheel_joint: axis 0 0 -1 -> 0 0 1; origin xyz=-0.100 -0.130 0 rpy=1.5707 0 0 -> xyz=0.136 0.130 0 rpy=-1.5707 0 0

Commit message: Add LRF

File: src/fifth_robot_description/fifth_robot.urdf (robot description, URDF)
Before this commit: robot fifth_robot, 5 links, 4 joints
Links:
- added link hokuyo_link, mass 1e-5; collision box size=0.1 0.1 0.1; visual box size=0.1 0.1 0.1
Joints:
- added joint hokuyo_joint: type fixed, parent base_link, child hokuyo_link, origin xyz=0.25 0 0.25 rpy=0 0 0, axis 0 0 1

Commit message: Fix URDF
吐き出しtopicを/scanにして扱いやすく, また, 返り値のよみができるように

File: src/fifth_robot_description/fifth_robot.urdf (robot description, URDF)
Before this commit: robot fifth_robot, 6 links, 5 joints
Links:
- link hokuyo_link: mass 1e-5 -> None; geometry visual box size=0.1 0.1 0.1
Joints:
- joint hokuyo_joint: axis 0 0 1 -> (none); origin xyz=0.25 0 0.25 rpy=0 0 0 -> xyz=0.1 0 0.1 rpy=0 0 0

Commit message: Amend wheel
逆でした, (滝汗)

File: src/fifth_robot_description/fifth_robot.urdf (robot description, URDF)
Before this commit: robot fifth_robot, 6 links, 5 joints
Joints:
- joint left_wheel_joint: origin xyz=0.136 -0.130 0 rpy=1.5707 0 0 -> xyz=0.136 0.130 0 rpy=1.5707 0 0
- joint right_wheel_joint: origin xyz=0.136 0.130 0 rpy=-1.5707 0 0 -> xyz=0.136 -0.130 0 rpy=-1.5707 0 0

Commit message: Enable double laser sim

File: src/fifth_robot_description/fifth_robot.urdf (robot description, URDF)
Before this commit: robot fifth_robot, 6 links, 5 joints
Links:
- removed link hokuyo_link
- added link front_hokuyo_link; visual box size=0.1 0.1 0.1
- added link rear_hokuyo_link; visual box size=0.1 0.1 0.1
Joints:
- added joint rear_hokuyo_joint: type fixed, parent base_link, child rear_hokuyo_link, origin xyz=-0.1 0 0.1 rpy=0 0 1.57
- joint hokuyo_joint: child hokuyo_link -> front_hokuyo_link

Commit message: Re:Fix rotate

File: src/fifth_robot_description/fifth_robot.urdf (robot description, URDF)
Before this commit: robot fifth_robot, 7 links, 6 joints
Joints:
- joint rear_hokuyo_joint: origin xyz=-0.1 0 0.1 rpy=0 0 1.57 -> xyz=-0.1 0 0.1 rpy=0 0 3.14
