Commit message: Remove rear sensor from urdf

File: src/fifth_robot_pkgs/fifth_robot_description/fifth_robot.urdf (robot description, URDF)
Before this commit: robot fifth_robot, 7 links, 6 joints
Links:
- removed link rear_hokuyo_link
Joints:
- removed joint rear_hokuyo_joint

Commit message: Rename 'front_hokuyo' => 'velodyne' in urdf

File: src/fifth_robot_pkgs/fifth_robot_description/fifth_robot.urdf (robot description, URDF)
Before this commit: robot fifth_robot, 6 links, 5 joints
Links:
- removed link front_hokuyo_link
- added link velodyne_link; visual box size=0.1 0.1 0.1
Joints:
- removed joint hokuyo_joint
- added joint velodyne_joint: type fixed, parent base_link, child velodyne_link, origin xyz=0 0 0.1 rpy=0 0 0

Commit message: Modify urdf to add imu link on gazebo

File: src/fifth_robot_pkgs/fifth_robot_description/fifth_robot.urdf (robot description, URDF)
Before this commit: robot fifth_robot, 6 links, 5 joints
Links:
- added link imu_link; visual box size=0.1 0.1 0.1
Joints:
- added joint imu_joint: type fixed, parent base_link, child imu_link, origin xyz=0 0.1 0.1 rpy=0 0 0

Commit message: Refactor gazebo model around imu sensor

File: src/fifth_robot_pkgs/fifth_robot_description/fifth_robot.urdf (robot description, URDF)
Before this commit: robot fifth_robot, 7 links, 6 joints
Links:
- link imu_link: geometry visual box size=0.02 0.02 0.02
Joints:
- joint imu_joint: origin xyz=0 0.1 0.1 rpy=0 0 0 -> xyz=0.15 0 0 rpy=0 0 0

Commit message: Fix position of joint of imu link

File: src/fifth_robot_pkgs/fifth_robot_description/fifth_robot.urdf (robot description, URDF)
Before this commit: robot fifth_robot, 7 links, 6 joints
Joints:
- joint imu_joint: origin xyz=0.15 0 0 rpy=0 0 0 -> xyz=0.16 0 0 rpy=0 0 0

Commit message: Remove link named base_footprint

File: src/fifth_robot_pkgs/fifth_robot_description/fifth_robot.urdf (robot description, URDF)
Before this commit: robot fifth_robot, 7 links, 6 joints
Links:
- removed link base_footprint
Joints:
- removed joint base_link_joint
