Commit message: Modify urdf to adjust to real machine

File: src/fifth_robot_pkgs/fifth_robot_description/config/controller/fifth_robot.urdf (robot description, URDF)
Before this commit: robot fifth_robot, 6 links, 5 joints
Links:
- link base_link: geometry collision box size=0.300 0.250 0.10; visual box size=0.300 0.250 0.20
Joints:
- joint velodyne_joint: origin xyz=0 0 0.1 rpy=0 0 0 -> xyz=0.1 0 0.2 rpy=0 0 0

Commit message: Adjust LiDAR height to real machine

File: src/fifth_robot_pkgs/fifth_robot_description/config/controller/fifth_robot.urdf (robot description, URDF)
Before this commit: robot fifth_robot, 6 links, 5 joints
Joints:
- joint velodyne_joint: origin xyz=0.1 0 0.2 rpy=0 0 0 -> xyz=0.1 0 0.7 rpy=0 0 0
